Commit message: Fixed swapped x and y axes

File: assets/gantry.urdf (robot description, URDF)
Before this commit: robot compact_gantry, 7 links, 6 joints
Links:
- link bridge_link: geometry visual box size=0.2 1.4 0.1
Joints:
- joint slider_x: axis 0 1 0 -> 1 0 0
- joint slider_y: axis 1 0 0 -> 0 1 0

Commit message: vision work

File: assets/gantry.urdf (robot description, URDF)
Before this commit: robot compact_gantry, 7 links, 6 joints
Links:
- added link bridge_cam, mass 0.05; visual box size=0.08 0.04 0.04
- added link wrist_cam, mass 0.05; visual box size=0.06 0.04 0.04
Joints:
- added joint bridge_cam_fixed: type fixed, parent bridge_link, child bridge_cam, origin xyz=-0.1 0.0 0.0 rpy=0 0 0
- added joint wrist_cam_fixed: type fixed, parent ee_link, child wrist_cam, origin xyz=0.0 0.0 -0.08 rpy=0 0 0

Commit message: nothing new

File: assets/gantry.urdf (robot description, URDF)
Before this commit: robot compact_gantry, 9 links, 8 joints
Joints:
- joint bridge_cam_fixed: origin xyz=-0.1 0.0 0.0 rpy=0 0 0 -> xyz=-0.1 0.5 0.0 rpy=-0.2 0 0
